File: schema/footie/V1.3.1/board.sch (EAGLE design)
At the start: 44 parts, among them T1 2N3565, U1 IRLML2246TRPBF, U2 USD-SOCKETNEW, U3 HC_05, U4 MCP73831, U5 3.3 regulator, U6 ATMEGA328P-AU

Commit message: finished route pcb expect antenna
Other:
- moved on the sheet: C2
Changed lines of the file:
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@@
 <instance part="GND23" gate="1" x="307.34" y="147.32"/>
 <instance part="GND24" gate="1" x="314.96" y="142.24"/>
-<instance part="GND25" gate="1" x="325.12" y="144.78"/>
+<instance part="GND25" gate="1" x="325.12" y="139.7"/>
 <instance part="P+1" gate="VCC" x="335.28" y="157.48" rot="R270"/>
 <instance part="BATTERY_CONNECTOR" gate="G$1" x="233.68" y="93.98"/>
@@
 <instance part="C3" gate="G$1" x="309.88" y="93.98"/>
 <instance part="C4" gate="G$1" x="264.16" y="88.9"/>
-<instance part="C2" gate="G$1" x="325.12" y="149.86"/>
+<instance part="C2" gate="G$1" x="325.12" y="147.32"/>
 <instance part="C8" gate="G$1" x="266.7" y="147.32"/>
 <instance part="LED2" gate="G$1" x="20.32" y="68.58" rot="R180"/>
@@
 <wire x1="304.8" y1="157.48" x2="325.12" y2="157.48" width="0.1524" layer="91"/>
 <wire x1="325.12" y1="157.48" x2="332.74" y2="157.48" width="0.1524" layer="91"/>
-<wire x1="325.12" y1="154.94" x2="325.12" y2="157.48" width="0.1524" layer="91"/>
+<wire x1="325.12" y1="152.4" x2="325.12" y2="157.48" width="0.1524" layer="91"/>
 <junction x="325.12" y="157.48"/>
 <pinref part="P+1" gate="VCC" pin="VCC"/>
@@
 <pinref part="GND25" gate="1" pin="GND"/>
 <pinref part="C2" gate="G$1" pin="2"/>
+<wire x1="325.12" y1="142.24" x2="325.12" y2="144.78" width="0.1524" layer="91"/>
 </segment>
 <segment>
@@
 </sheet>
 </sheets>
-<errors>
-</errors>
 </schematic>
 </drawing>

Commit message: complete the board layout
Parts:
- BATTERY_CONNECTOR, BLUETOOTH, DEBUG, GPS_ANTENNA, JP2, MICRO_USB, U$1: OC_FARNELL (none) -> unknown
- C1, C5, C6: MF (none) -> KEMET; MPN (none) -> C0402C104K4RACTU; OC_FARNELL (none) -> 1288252
- C10, C11: MF (none) -> MULTICOMP; MPN (none) -> MC1206F226Z100CT; OC_FARNELL (none) -> 1759435
- C2, C8, C9: MF (none) -> WALSIN; MPN (none) -> 1206B475K500CT; OC_FARNELL (none) -> 2497114
- C3, C4: MF (none) -> WALSIN; MPN (none) -> 1206B106K160CT; OC_FARNELL (none) -> 2497081
- CHARGING, GPS_STATUS: MF (none) -> KINGBRIGHT; MPN (none) -> KPTL-3216ZGC; OC_FARNELL (none) -> 2217899
- D1: MF (none) -> VISHAY; MPN (none) -> BZG03C18TR3; OC_FARNELL (none) -> 9398112
- LED_STATUS: MF (none) -> AVAGO TECHNOLOGIES; MPN (none) -> ASMB-MTB0-0A3A2; OC_FARNELL (none) -> 2401105
- POWER: value (none) -> red; MF (none) -> KINGBRIGHT; MPN (none) -> KPTL-3216SURCK-01; OC_FARNELL (none) -> 2217903
- Q2: MF (none) -> ABRACON; MPN (none) -> ABMM2-8.000MHZ-E2-T; OC_FARNELL (none) -> 1611803
- R1: MF (none) -> YAGEO (PHYCOMP); MPN (none) -> RC1206FR-07100RL; OC_FARNELL (none) -> 9240888
- R10, R11, R12, R2, R5, R6, R7: MF (none) -> VISHAY; MPN (none) -> CRCW12061K00FKTA; OC_FARNELL (none) -> 1653075
- R3, R4: MF (none) -> VISHAY; MPN (none) -> CRCW120610K0FKEA; OC_FARNELL (none) -> 1469970
- R8: MF (none) -> WELWYN; MPN (none) -> WCR1206-330RFI; OC_FARNELL (none) -> 1100177
- R9: MF (none) -> VISHAY; MPN (none) -> CRCW12062K00FKEA; OC_FARNELL (none) -> 1469985
- S_MODE, S_TRACK: MF (none) -> TE CONNECTIVITY; MPN (none) -> FSM1LP; OC_FARNELL unknown -> 1813691
- T1: MF (none) -> ON SEMICONDUCTOR; MPN (none) -> 2N5089G; OC_FARNELL (none) -> 1126530
- U$3: MF (none) -> SEIKO INSTRUMENTS; MPN (none) -> MS621FE-FL11E; OC_FARNELL (none) -> 1614634
- U1: MF (none) -> INFINEON
- U2: MF (none) -> MULTICOMP; MPN (none) -> 460DE08C3; OC_FARNELL (none) -> 1686452
- U4: MF (none) -> MICROCHIP; MPN (none) -> MCP73831T-2ACI/OT; OC_FARNELL (none) -> 1332158
- U5: MF (none) -> MICREL SEMICONDUCTOR; MPN (none) -> MIC5205-3.3YM5 TR; OC_FARNELL (none) -> 1663083
- U6: MF (none) -> ATMEL
- renumbered LED2 to GPS_STATUS, LED3 to LED_STATUS, LED4 to CHARGING, LED5 to POWER, U$2 to DEBUG, U3 to BLUETOOTH

Commit message: complete board but not happy
Parts:
- removed GPS_ANTENNA: ANTENNA2SMD6, SparkFun-RF:ANTENNA2SMD6
- removed U$1: UBLOX_NEO-6, Ava:UBLOX_NEO-6
- added C7: 4.7 uF, SparkFun-Capacitors:CAP1206
- added R13, R14: 220 Ohm, SparkFun-Passives:RESISTOR1206
- added U3: CAM-M8Q, CAM-M8Q:CAM-M8Q
Connections:
- removed net N$6 (its old number): R2.1, U$1.22_V_BCKP, U$3.3V
- removed net N$7: GPS_ANTENNA.SIGNAL, U$1.11_RF_IN
- removed net SCL: U$1.19_SCL2
- removed net SDA: U$1.18_SDA2
- new net N$25: R13.1, U3.TXD
- new net N$26: R14.1, U3.RXD
- new net N$4: R6.2, U3.TIMEPULSE
- net +3V3: now also C7.1, U3.VCC, U3.VCC_IO; no longer U$1.23_VCC
- net GND: now also C7.2, U3.GND@1, U3.GND@10, U3.GND@11, U3.GND@12, U3.GND@13, U3.GND@14, U3.GND@2, U3.GND@3, U3.GND@4, U3.GND@5, U3.GND@6, U3.GND@7, U3.GND@8, U3.GND@9; no longer U$1.10_GND, U$1.12_GND, U$1.13_GND, U$1.24_GND, U$1.7_VDDUSB
- net GPSRX: now also R14.2; no longer U$1.21_RXD1
- net GPSTX: now also R13.2; no longer U$1.20_TXD1
- net N$3: now also U3.ANT, U3.RF_IN; no longer R6.2, U$1.3_TIMEPULSE
- net N$5: now also R2.1, U$3.3V, U3.V_BCKP; no longer U$1.8_RESERVED, U$1.9_VCC_RF
Other:
- moved on the sheet: D1, GPS_STATUS, R2, R6

Commit message: update final version + library
Parts:
- S_MODE: value DTSM-6 -> MODE
- S_TRACK: value DTSM-6 -> TRACK
Connections:
- net GND: no longer BLUETOOTH.GND1, BLUETOOTH.GND2
- net N$20: now also BLUETOOTH.GND1, BLUETOOTH.GND2
Changed lines of the file:
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@@
 </classes>
 <parts>
-<part name="S_MODE" library="switch-tact" deviceset="DTSM-6" device="">
+<part name="S_MODE" library="switch-tact" deviceset="DTSM-6" device="" value="MODE">
 <attribute name="MF" value="TE CONNECTIVITY"/>
 <attribute name="MPN" value="FSM1LP"/>
 <attribute name="OC_FARNELL" value="1813691"/>
 </part>
-<part name="S_TRACK" library="switch-tact" deviceset="DTSM-6" device="">
+<part name="S_TRACK" library="switch-tact" deviceset="DTSM-6" device="" value="TRACK">
 <attribute name="MF" value="TE CONNECTIVITY"/>
 <attribute name="MPN" value="FSM1LP"/>
@@
 </part>
 <part name="+3V7" library="supply1" deviceset="+3V3" device=""/>
-<part name="GND16" library="supply1" deviceset="GND" device=""/>
-<part name="GND17" library="supply1" deviceset="GND" device=""/>
 <part name="U4" library="SparkFun-PowerIC" deviceset="MCP73831" device="">
 <attribute name="MF" value="MICROCHIP"/>
@@
 </instance>
 <instance part="+3V7" gate="G$1" x="264.16" y="20.32" rot="R90"/>
-<instance part="GND16" gate="1" x="309.88" y="7.62" rot="MR0"/>
-<instance part="GND17" gate="1" x="327.66" y="17.78" rot="MR270"/>
 <instance part="U4" gate="G$1" x="294.64" y="154.94">
 <attribute name="OC_FARNELL" x="294.64" y="154.94" size="1.778" layer="96" display="off"/>
@@
 <wire x1="279.4" y1="17.78" x2="276.86" y2="17.78" width="0.1524" layer="91"/>
 <wire x1="276.86" y1="17.78" x2="274.32" y2="17.78" width="0.1524" layer="91"/>
-<wire x1="274.32" y1="17.78" x2="274.32" y2="10.16" width="0.1524" layer="91"/>
+<wire x1="274.32" y1="17.78" x2="274.32" y2="12.7" width="0.1524" layer="91"/>
 <junction x="274.32" y="10.16"/>
 <junction x="279.4" y="17.78"/>
 <pinref part="BLUETOOTH" gate="G$1" pin="GND"/>
 <junction x="276.86" y="17.78"/>
+<pinref part="BLUETOOTH" gate="G$1" pin="GND1"/>
+<wire x1="274.32" y1="12.7" x2="274.32" y2="10.16" width="0.1524" layer="91"/>
+<wire x1="309.88" y1="10.16" x2="309.88" y2="5.08" width="0.1524" layer="91"/>
+<wire x1="309.88" y1="5.08" x2="279.4" y2="5.08" width="0.1524" layer="91"/>
+<wire x1="279.4" y1="5.08" x2="279.4" y2="12.7" width="0.1524" layer="91"/>
+<wire x1="279.4" y1="12.7" x2="274.32" y2="12.7" width="0.1524" layer="91"/>
+<junction x="274.32" y="12.7"/>
+<pinref part="BLUETOOTH" gate="G$1" pin="GND2"/>
+<wire x1="325.12" y1="17.78" x2="330.2" y2="17.78" width="0.1524" layer="91"/>
+<wire x1="330.2" y1="17.78" x2="330.2" y2="5.08" width="0.1524" layer="91"/>
+<wire x1="330.2" y1="5.08" x2="309.88" y2="5.08" width="0.1524" layer="91"/>
+<junction x="309.88" y="5.08"/>
 </segment>
 </net>
@@
 </segment>
 <segment>
-<pinref part="BLUETOOTH" gate="G$1" pin="GND1"/>
-<pinref part="GND16" gate="1" pin="GND"/>
-</segment>
-<segment>
-<pinref part="BLUETOOTH" gate="G$1" pin="GND2"/>
-<pinref part="GND17" gate="1" pin="GND"/>
-</segment>
-<segment>

Commit message: update stuff2
Parts:
- C7: MPN 1206B106K160CT -> 1206B475K500CT; OC_FARNELL 2497081 -> 2497114
- U3: OC_FARNELL (none) -> unknown
Connections:
- net +3V3: now also LED_STATUS.ANODE
- net GND: no longer LED_STATUS.ANODE
Changed lines of the file:
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@@
 </part>
 <part name="+3V13" library="supply1" deviceset="+3V3" device=""/>
-<part name="GND8" library="supply1" deviceset="GND" device=""/>
 <part name="U1" library="pretender" deviceset="IRLML2246TRPBF" device="">
 <attribute name="MF" value="INFINEON"/>
@@
 <attribute name="OC_FARNELL" value="1653075"/>
 </part>
-<part name="U3" library="CAM-M8Q" deviceset="CAM-M8Q" device=""/>
+<part name="U3" library="CAM-M8Q" deviceset="CAM-M8Q" device="">
+<attribute name="MF" value=""/>
+<attribute name="MPN" value=""/>
+<attribute name="OC_FARNELL" value="unknown"/>
+</part>
 <part name="GND9" library="supply1" deviceset="GND" device=""/>
 <part name="GND15" library="supply1" deviceset="GND" device=""/>
@@
 <part name="C7" library="SparkFun-Capacitors" deviceset="CAP" device="1206" value="4.7 uF">
 <attribute name="MF" value="WALSIN"/>
-<attribute name="MPN" value="1206B106K160CT"/>
-<attribute name="OC_FARNELL" value="2497081"/>
-</part>
+<attribute name="MPN" value="1206B475K500CT"/>
+<attribute name="OC_FARNELL" value="2497114"/>
+</part>
+<part name="+3V1" library="supply1" deviceset="+3V3" device=""/>
 </parts>
 <sheets>
@@
 </instance>
 <instance part="+3V13" gate="G$1" x="157.48" y="134.62" rot="R270"/>
-<instance part="GND8" gate="1" x="7.62" y="170.18" rot="R180"/>
 <instance part="U1" gate="A" x="251.46" y="91.44" rot="R90">
 <attribute name="MF" x="251.46" y="91.44" size="1.778" layer="96" display="off"/>
@@
 <attribute name="MPN" x="-2.54" y="147.32" size="1.778" layer="96" display="off"/>
 </instance>
-<instance part="U3" gate="G$1" x="63.5" y="88.9"/>
+<instance part="U3" gate="G$1" x="63.5" y="88.9">
+<attribute name="OC_FARNELL" x="63.5" y="88.9" size="1.778" layer="96" display="off"/>
+<attribute name="MF" x="63.5" y="88.9" size="1.778" layer="96" display="off"/>
+<attribute name="MPN" x="63.5" y="88.9" size="1.778" layer="96" display="off"/>
+</instance>
 <instance part="GND9" gate="1" x="48.26" y="60.96" rot="R270"/>
 <instance part="GND15" gate="1" x="76.2" y="60.96" rot="R90"/>
@@
 <attribute name="MPN" x="142.24" y="93.98" size="1.778" layer="96" display="off"/>
 </instance>
+<instance part="+3V1" gate="G$1" x="7.62" y="172.72"/>
 </instances>
 <busses>
@@
 <pinref part="D1" gate="D" pin="A"/>
 <junction x="114.3" y="96.52"/>
+</segment>
+<segment>
+<pinref part="LED_STATUS" gate="A" pin="ANODE"/>
+<pinref part="+3V1" gate="G$1" pin="+3V3"/>
+<wire x1="7.62" y1="167.64" x2="7.62" y2="170.18" width="0.1524" layer="91"/>
 </segment>
 </net>
@@
 </segment>
 <segment>
-<pinref part="GND8" gate="1" pin="GND"/>
-<pinref part="LED_STATUS" gate="A" pin="ANODE"/>
-<junction x="7.62" y="167.64"/>
-</segment>
-<segment>
