File: schema/footie/V1.3.2/board.sch (EAGLE design)
At the start: 41 parts, among them T1 2N3565, U1 IRLML2246TRPBF, U2 USD-SOCKETNEW, U4 MCP73831, U5 3.3 regulator, U6 ATMEGA328P-AU

Commit message: update parser fix schematic wiring
Connections:
- net ARDUINO_RX: now also JP1.5; no longer JP1.4
- net ARDUINO_TX: now also JP1.4; no longer JP1.5
Changed lines of the file:
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@@
 </segment>
 <segment>
-<wire x1="86.36" y1="81.28" x2="63.5" y2="81.28" width="0.1524" layer="91"/>
-<label x="86.36" y="83.82" size="1.778" layer="95" rot="R180"/>
-<pinref part="JP1" gate="G$1" pin="5"/>
-<wire x1="63.5" y1="91.44" x2="63.5" y2="81.28" width="0.1524" layer="91"/>
+<label x="86.36" y="78.74" size="1.778" layer="95" rot="R180"/>
+<pinref part="JP1" gate="G$1" pin="4"/>
+<wire x1="60.96" y1="91.44" x2="60.96" y2="76.2" width="0.1524" layer="91"/>
+<wire x1="60.96" y1="76.2" x2="86.36" y2="76.2" width="0.1524" layer="91"/>
 </segment>
 </net>
@@
 </segment>
 <segment>
-<label x="86.36" y="78.74" size="1.778" layer="95" rot="R180"/>
-<pinref part="JP1" gate="G$1" pin="4"/>
-<wire x1="60.96" y1="91.44" x2="60.96" y2="76.2" width="0.1524" layer="91"/>
-<wire x1="60.96" y1="76.2" x2="86.36" y2="76.2" width="0.1524" layer="91"/>
+<wire x1="86.36" y1="81.28" x2="63.5" y2="81.28" width="0.1524" layer="91"/>
+<label x="86.36" y="83.82" size="1.778" layer="95" rot="R180"/>
+<pinref part="JP1" gate="G$1" pin="5"/>
+<wire x1="63.5" y1="91.44" x2="63.5" y2="81.28" width="0.1524" layer="91"/>
 </segment>
 </net>
